Commit message: Fixed xacro file and increased particle count.

File: src/my_robot/urdf/my_robot.xacro (robot description, xacro)
@@ -68,5 +68,5 @@
   </link>
   <joint type="continuous" name="left_wheel_hinge">
-    <origin xyz="-0.1 -0.13 0" rpy="0 0 0"/>
+    <origin xyz="-0.1 0.13 0" rpy="0 0 0"/>
     <child link="left_wheel"/>
     <parent link="chassis"/>
@@ -99,5 +99,5 @@
   </link>
   <joint type="continuous" name="right_wheel_hinge">
-    <origin xyz="-0.1 0.13 0" rpy="0 0 0"/>
+    <origin xyz="-0.1 -0.13 0" rpy="0 0 0"/>
     <child link="right_wheel"/>
     <parent link="chassis"/>

Commit message: Fixed configs and refactor robot xacro to be dimensions specified in first project.

File: src/my_robot/urdf/my_robot.xacro (robot description, xacro)
@@ -22,5 +22,5 @@
       <origin xyz="0 0 0" rpy=" 0 0 0"/>
       <geometry>
-        <box size=".5 .2 .1"/>
+        <box size=".4 .2 .1"/>
       </geometry>
     </collision>
@@ -28,11 +28,23 @@
       <origin xyz="0 0 0" rpy=" 0 0 0"/>
       <geometry>
-        <box size=".5 .2 .1"/>
+        <box size=".4 .2 .1"/>
+      </geometry>
+    </visual>
+    <collision name='back_caster_collision'>
+      <origin xyz="-0.15 0 -0.05" rpy=" 0 0 0"/>
+      <geometry>
+        <sphere radius="0.05"/>
+      </geometry>
+    </collision>
+    <visual name='back_caster_visual'>
+      <origin xyz="-0.15 0 -0.05" rpy=" 0 0 0"/>
+      <geometry>
+        <sphere radius="0.05"/>
       </geometry>
     </visual>
     <collision name='front_caster_collision'>
-      <origin xyz="0.2 0 -0.05" rpy=" 0 0 0"/>
+      <origin xyz="0.15 0 -0.05" rpy=" 0 0 0"/>
       <geometry>
-        <sphere radius="0.02"/>
+        <sphere radius="0.05"/>
       </geometry>
     </collision>
@@ -40,5 +52,5 @@
       <origin xyz="0.15 0 -0.05" rpy=" 0 0 0"/>
       <geometry>
-        <sphere radius="0.02"/>
+        <sphere radius="0.05"/>
       </geometry>
     </visual>
@@ -57,5 +69,5 @@
       <origin xyz="0 0 0 " rpy=" 0 1.5707 1.5707"/>
         <geometry>
-          <cylinder radius="0.07" length="0.05"/>
+          <cylinder radius="0.1" length="0.05"/>
         </geometry>
     </collision>
@@ -63,10 +75,10 @@
       <origin xyz="0 0 0 " rpy=" 0 1.5707 1.5707"/>
         <geometry>
-          <cylinder radius="0.07" length="0.05"/>
+          <cylinder radius="0.1" length="0.05"/>
         </geometry>
     </visual>
   </link>
   <joint type="continuous" name="left_wheel_hinge">
-    <origin xyz="-0.1 0.13 0" rpy="0 0 0"/>
+    <origin xyz="0 0.15 0" rpy="0 0 0"/>
     <child link="left_wheel"/>
     <parent link="chassis"/>
@@ -88,5 +100,5 @@
       <origin xyz="0 0 0 " rpy=" 0 1.5707 1.5707"/>
         <geometry>
-          <cylinder radius="0.07" length="0.05"/>
+          <cylinder radius="0.1" length="0.05"/>
         </geometry>
     </collision>
@@ -94,10 +106,10 @@
       <origin xyz="0 0 0 " rpy=" 0 1.5707 1.5707"/>
         <geometry>
-          <cylinder radius="0.07" length="0.05"/>
+          <cylinder radius="0.1" length="0.05"/>
         </geometry>
     </visual>
   </link>
   <joint type="continuous" name="right_wheel_hinge">
-    <origin xyz="-0.1 -0.13 0" rpy="0 0 0"/>
+    <origin xyz="0 -0.15 0" rpy="0 0 0"/>
     <child link="right_wheel"/>
     <parent link="chassis"/>
@@ -131,5 +143,5 @@
   </link>
   <joint type="fixed" name="camera_joint">
-    <origin xyz="0.25 0 0" rpy="0 0 0"/>
+    <origin xyz="0.2 0 0" rpy="0 0 0"/>
     <child link="camera"/>
     <parent link="chassis"/>
@@ -160,5 +172,5 @@
   </link>
   <joint type="fixed" name="hokuyo_joint">
-    <origin xyz="0.15 0 0.07" rpy="0 0 0"/>
+    <origin xyz="0.15 0 0.1" rpy="0 0 0"/>
     <child link="hokuyo"/>
     <parent link="chassis"/>

Commit message: Reduced collision size of casters on robot as they were adding friction and causing the robot to drive incorrectly. Increased the amcl configs for performing updates.

File: src/my_robot/urdf/my_robot.xacro (robot description, xacro)
@@ -34,5 +34,5 @@
       <origin xyz="-0.15 0 -0.05" rpy=" 0 0 0"/>
       <geometry>
-        <sphere radius="0.05"/>
+        <sphere radius="0.0499"/>
       </geometry>
     </collision>
@@ -46,5 +46,5 @@
       <origin xyz="0.15 0 -0.05" rpy=" 0 0 0"/>
       <geometry>
-        <sphere radius="0.05"/>
+        <sphere radius="0.0499"/>
       </geometry>
     </collision>
